File: Hardware/9DOF-Razor-v23.sch (EAGLE design)
At the start: 41 parts, among them J1 AVR_SPI_PRG_6PTH, Q1 8MHz, U1 ITG-32001:1, U2 ADXL3451:1, U5 3.3V, U6 ATMEGA328

Commit message: General cleanup in schematic
Added:
- Rev code on PCB
- Minor trace cleanup on mag IC
Replaced:
- Net labels with flag style markers
- Old Frame design with new Frame design that includes CC3.0 and OSHW
stuff
Parts:
- removed U$3: CREATIVE_COMMONS, SparkFun:CREATIVE_COMMONS
Other:
- note added: "Kade Alexander Jensen"
- note removed: "Kade Jensen"
